File: hardware/pdm-hc2/ESP32-PDM-HC2.kicad_sch (KiCad schematic)
At the start: 19 parts, among them J10 POWER, J11 OUTPUTS, U1 ESP32-S3-MINI-1

Commit message: System: panel cable and pin map – fused switch supply, MMBT5551 LED sinks, VBAT and NTC (decisions 17-21)
Co-Authored-By: Claude Opus 5.5 <noreply@anthropic.com>
Parts:
- added C60, C61: 100nF, Capacitor_SMD:C_0402_1005Metric, symbol Device:C
- added R60: 220k, Resistor_SMD:R_0402_1005Metric, symbol Device:R
- added R61: 22k, Resistor_SMD:R_0402_1005Metric, symbol Device:R
- added R62: 10k, Resistor_SMD:R_0402_1005Metric, symbol Device:R
- added TH1: 10k B3380, Resistor_SMD:R_0603_1608Metric, symbol Device:Thermistor_NTC
Connections:
- net +3V3: now also R62.1
- net GND: now also C60.2, C61.2, R61.2, TH1.2
- net IO11: now also R2.2
- net VS: now also R60.1
- net IO38: now reaches U1.34 (IO38)
- net IO39: now reaches U1.35 (IO39)
- net IO40: now reaches U1.36 (IO40)
- net IO41: now reaches U1.37 (IO41)
- net IO10 renamed VBAT_SENSE
- net VBAT_SENSE: now also C60.1, R60.2, R61.1
- net IO12: no longer names the net of U1.16 (IO12)
- net IO13: no longer names the net of U1.17 (IO13)
- net IO9 renamed NTC
- net NTC: now also C61.1, R62.2, TH1.1; no longer R2.2
- no-connect marks 15 -> 13
Other:
- note added: "Decision 18: VBAT_SENSE on IO10 (ADC1): 220k/22k, 33 V full scale. NTC on IO9 (ADC1): 10k pull-up, TH1 next to the output switches. Panel LED drives on IO38-IO41 (sheet pins DIAG1-4)."
- note added: "Spare GPIO: IO4, IO5, IO8, IO12, IO13, IO26, IO33, IO42, IO45-IO48 (no-connect flags; IO45/IO46 are strapping pins; IO8/IO11 keep 2.2k pull-downs R1/R2)"
- note removed: "Spare GPIO: IO4, IO5, IO26, IO33, IO38-IO42, IO45-IO48 (no-connect flags; IO45/IO46 are strapping pins)"
